File: Moteur.kicad_pcb (KiCad board)
At the start: 4 copper layers, 31.7 x 16.1 mm, 53 parts, among them IC1 TPS71501, IC2 TLV710, IC3 MAX3051, IC4 LM5106, IC5 LM5106, IC6 INA282, P1 Bus2, P2 MOTOR, P3 GPIO, P4 CONN_1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

Commit message: routing
Parts:
- moved R5 7.01 mm to (130.9, 101.0), turned to 0 degrees
- moved R3 6.41 mm to (130.9, 99.8), turned to 0 degrees
- moved R6 6.11 mm to (130.9, 102.3)
- moved C5 1.45 mm to (128.8, 97.3)
- moved R9 0.45 mm to (137.6, 97.9)
- moved C15 0.41 mm to (137.6, 96.6)
- moved C17 0.30 mm to (126.2, 103.2)
- moved R1 0.30 mm to (140.9, 99.4)
- moved C10 0.25 mm to (127.5, 99.8)
- moved C8 0.14 mm to (135.8, 100.8)
Connections:
- IC4 pad 7: Mot_En_1 -> Mot_En_2
- IC4 pad 8: PWM1 -> PWM2
- IC5 pad 7: Mot_En_2 -> Mot_En_1
- IC5 pad 8: PWM2 -> PWM1
- P3 pad 1: GPIO_ADC -> I
- P3 pad 2: I -> GPIO_B
- P3 pad 3: GPIO_B -> GPIO_A
- P3 pad 4: GPIO_A -> GPIO_ADC
- P3 pad 5: GND -> +3.3V_A
- P3 pad 6: +3.3V_A -> GND
Routing:
- net +5V_protected: track 5.97 -> 31.2 mm
- net B: track 1.87 -> 22.7 mm
- net A: track 0.00 -> 20.8 mm, vias 0 -> 1
- net Mot_En_1: track 1.71 -> 18.3 mm, vias 1 -> 2
- net PWM1: track 1.54 -> 15.4 mm, vias 1 -> 2
- net Mot_En_2: track 1.14 -> 15.0 mm, vias 1 -> 2
- net Tx: track 2.41 -> 14.6 mm
- net Rx: track 2.05 -> 13.8 mm
- net PWM2: track 1.50 -> 12.7 mm, vias 1 -> 2
- net +9V: track 3.86 -> 14.9 mm, vias 0 -> 1
- net +BATT: track 13.4 -> 22.3 mm
- net ADC/I_MOT: track 7.31 -> 0.00 mm
- net Swdio: track 9.08 -> 2.35 mm
- net N-0000043: track 0.00 -> 5.90 mm
- net GPIO_A: track 0.00 -> 4.63 mm
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
Commit message: routing
Parts:
- added C19: 100nF (DNP), _0603, B.Cu at (140.3, 91.4)
- moved R3 11.5 mm to (119.7, 102.0)
- moved L1 9.27 mm to (126.5, 100.0), turned to 0 degrees
- moved C8 2.45 mm to (134.9, 103.1), turned to 180 degrees
- moved R5 1.89 mm to (129.4, 102.2)
- moved C10 1.63 mm to (128.6, 98.5)
- moved R6 1.52 mm to (132.2, 103.0)
- moved C5 0.74 mm to (128.6, 96.7)
Routing:
- net +5V_protected: track 31.2 -> 8.20 mm
- net ADC/I_MOT: track 0.00 -> 13.3 mm, vias 0 -> 1
- net N-0000040: track 0.00 -> 12.3 mm, vias 0 -> 2
- net +3.3V_A: track 10.0 -> 21.7 mm, vias 0 -> 1
- net I: track 3.04 -> 13.5 mm
- net GPIO_B: track 1.78 -> 11.9 mm
- net GPIO_A: track 4.63 -> 12.6 mm, vias 0 -> 1
- net GND: track 16.6 -> 23.5 mm, vias 1 -> 4
- net Swdio: track 2.35 -> 9.12 mm
- net GPIO_ADC: track 0.00 -> 6.11 mm, vias 0 -> 1
- net CAN_SPEED: track 15.5 -> 17.3 mm, vias 1 -> 2
- net +9V: track 14.9 -> 16.6 mm
- net +3.3V: track 19.8 -> 18.5 mm
- net N-0000038: track 7.50 -> 8.73 mm
- net Reset: track 10.6 -> 11.7 mm
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
Commit message: routing
Parts:
- moved R3 9.76 mm to (129.4, 102.4)
- moved R6 2.30 mm to (134.6, 103.0)
- moved R5 2.17 mm to (131.6, 102.5), turned to 270 degrees
- moved C8 1.76 mm to (136.7, 102.7), turned to 270 degrees
- moved L1 1.50 mm to (128.1, 100.0)
- moved C6 0.81 mm to (128.1, 93.7), turned to 90 degrees
- moved C13 0.74 mm to (130.5, 94.2)
- moved C11 0.45 mm to (126.2, 95.0)
Routing:
- net GND: track 23.5 -> 38.7 mm, vias 4 -> 8
- net +5V_protected: track 8.20 -> 20.9 mm, vias 0 -> 1
- net N-0000044: track 21.6 -> 31.6 mm, vias 0 -> 2
- net +3.3V: track 18.5 -> 27.4 mm
- net +3.3V_A: track 21.7 -> 28.5 mm
- net GPIO_A: track 12.6 -> 15.8 mm
- net GPIO_B: track 11.9 -> 14.8 mm
- net Mot+: track 18.1 -> 20.7 mm
- net I: track 13.5 -> 15.4 mm
- net Tx: track 14.9 -> 14.1 mm
- net ADC/I_MOT: track 13.3 -> 12.7 mm
- net ADC/V_BAT: track 14.2 -> 14.9 mm
- net N-0000040: track 12.3 -> 11.7 mm
Other:
- board size 31.7 x 16.1 mm -> 30.8 x 16.1 mm

Commit message: routing
Routing:
- net +5V_protected: track 20.9 -> 45.9 mm
- net GND: track 38.7 -> 46.5 mm
- net CAN_SPEED: track 17.3 -> 19.7 mm
- added copper zone on Inner2.Cu, net +3.3V
- added copper zone on B.Cu, net GND
- added copper zone on F.Cu, net GND
- added copper zone on Inner1.Cu, net GND
Other:
- board size 30.8 x 16.1 mm -> 30.8 x 16 mm

Commit message: routing
Parts:
- moved C9 1.04 mm to (137.6, 95.3), turned to 0 degrees
- moved C14 0.25 mm to (143.6, 98.5)
- moved C5 0.11 mm to (128.6, 96.8)
Connections:
- P3 pad 2: GPIO_B -> GPIO_A
- P3 pad 3: GPIO_A -> GPIO_B
- R3 pad 2: GPIO_A -> GPIO_B
- R5 pad 2: GPIO_B -> GPIO_A
Routing:
- net +3.3V: track 27.4 -> 49.5 mm, vias 4 -> 5
- net +5V_protected: track 45.9 -> 53.9 mm
- net Swdio: track 9.12 -> 11.7 mm
- net GND: track 46.5 -> 44.2 mm, vias 8 -> 9
- net N-0000044: track 31.6 -> 29.4 mm
- net Mot-: track 14.9 -> 12.8 mm
- net Rx: track 14.7 -> 16.3 mm
- net Tx: track 14.1 -> 15.1 mm
- net GPIO_A: track 15.8 -> 15.1 mm
- net Reset: track 12.0 -> 11.4 mm
- net Mot_En_2: track 14.2 -> 13.7 mm

Commit message: routing, almost done
Parts:
- moved C2 3.32 mm to (125.0, 101.7), turned to 180 degrees
- moved C3 2.83 mm to (125.8, 97.7)
- moved IC2 2.39 mm to (125.1, 99.7)
- moved R4 1.35 mm to (126.3, 101.5), turned to 180 degrees
- moved R3 0.81 mm to (130.2, 102.5), turned to 270 degrees
- moved C17 0.70 mm to (125.5, 103.2)
- moved D2 0.53 mm to (126.3, 102.8), turned to 180 degrees
- moved L1 0.50 mm to (128.6, 100.0)
- moved D1 0.10 mm to (123.5, 101.4)
Routing:
- net GND: track 44.2 -> 74.9 mm, vias 9 -> 12
- net N-0000044: track 29.4 -> 37.8 mm
- net +3.3V: track 49.5 -> 56.9 mm
- net Mot+: track 20.7 -> 26.4 mm
- net CAN_SPEED: track 19.7 -> 22.4 mm
- net N-0000064: track 4.03 -> 5.60 mm
- net +BATT: track 22.3 -> 23.6 mm
- net Rx: track 16.3 -> 15.4 mm
- net GPIO_B: track 14.9 -> 14.1 mm
- net Tx: track 15.1 -> 14.3 mm
- net +5V_protected: track 53.9 -> 54.5 mm
- added copper zone on Inner2.Cu, net GND

Commit message: routing, changed connectors
Parts:
- P4, P6: footprint _Pin2mm_2 -> PWR_Conn
- moved P4 1.23 mm to (151.8, 104.7)
- moved P6 1.22 mm to (151.8, 91.3)
Connections:
- P1 pad 1: CANH -> CANL
- P1 pad 2: CANL -> CANH
Routing:
- net GND: track 74.9 -> 91.7 mm
- net CANL: track 2.51 -> 5.91 mm
- net CANH: track 3.18 -> 2.44 mm
- net CAN_SPEED: track 22.4 -> 21.7 mm
