File: Moteur.sch (KiCad schematic (older format))
At the start: 53 parts, among them IC1 TPS71501, IC2 TLV710, IC3 MAX3051, IC4 LM5106, IC5 LM5106, IC6 INA282, P1 Bus2, P2 MOTOR, P3 GPIO, P4 CONN_1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

Commit message: routing
Other:
- moved on the sheet: P3, R3, R5, R6
Changed lines of the file:
@@
 Text GLabel 12750 5300 3    60   BiDi ~ 0
 Mot-
+Text GLabel 14800 3550 2    60   Input ~ 0
+PWM1
 Text GLabel 10500 3550 0    60   Input ~ 0
-PWM1
-Text GLabel 14800 3550 2    60   Input ~ 0
 PWM2
 $Comp
@@
 	-1   0    0    1
 $EndComp
+Text GLabel 14800 3350 2    60   Input ~ 0
+Mot_En_1
 Text GLabel 10500 3350 0    60   Input ~ 0
-Mot_En_1
-Text GLabel 14800 3350 2    60   Input ~ 0
 Mot_En_2
 Text GLabel 11850 5900 0    60   Input ~ 0
@@
 Text GLabel 3000 9150 2    60   Input ~ 0
 CANL
-Text GLabel 2250 7500 2    60   Input ~ 0
+Text GLabel 2300 7500 2    60   Input ~ 0
 I
 Text GLabel 1450 5600 2    60   Input ~ 0
@@
 	1    0    0    -1
 $EndComp
-Text GLabel 1500 7600 2    60   Input ~ 0
+Text GLabel 1350 7200 2    60   Input ~ 0
 GPIO_ADC
 $Comp
 L +3.3V_A #PWR11
 U 1 1 5464C7D0
-P 1550 7000
-F 0 "#PWR11" H 1550 6960 30  0001 C CNN
-F 1 "+3.3V_A" H 1550 7110 30  0000 C CNN
-F 2 "" H 1550 7000 60  0000 C CNN
-F 3 "" H 1550 7000 60  0000 C CNN
-	1    1550 7000
+P 1400 6950
+F 0 "#PWR11" H 1400 6910 30  0001 C CNN
+F 1 "+3.3V_A" H 1400 7060 30  0000 C CNN
+F 2 "" H 1400 6950 60  0000 C CNN
+F 3 "" H 1400 6950 60  0000 C CNN
+	1    1400 6950
 	1    0    0    -1
 $EndComp
@@
 L +5V_protected #PWR8
 U 1 1 5464CB8A
-P 1450 6900
-F 0 "#PWR8" H 1450 6990 20  0001 C CNN
-F 1 "+5V_protected" H 1450 6990 30  0000 C CNN
-F 2 "" H 1450 6900 60  0000 C CNN
-F 3 "" H 1450 6900 60  0000 C CNN
-	1    1450 6900
+P 1300 6800
+F 0 "#PWR8" H 1300 6890 20  0001 C CNN
+F 1 "+5V_protected" H 1300 6890 30  0000 C CNN
+F 2 "" H 1300 6800 60  0000 C CNN
+F 3 "" H 1300 6800 60  0000 C CNN
+	1    1300 6800
 	1    0    0    -1
 $EndComp
@@
 CANH
 Wire Wire Line
-	1500 7600 1450 7600
-Wire Wire Line
 	3350 4100 3350 4200
 Wire Wire Line
@@
 	4150 900  4150 950
 Wire Wire Line
-	1450 7500 2250 7500
+	1300 7500 2300 7500
 Wire Wire Line
 	4350 5950 4350 6100
@@
 	1450 9000 1500 9000
 Wire Wire Line
-	1450 7400 2250 7400
-Wire Wire Line
-	1450 7300 2250 7300
+	1300 7400 2300 7400
+Wire Wire Line
+	1300 7300 2300 7300
 Wire Wire Line
 	2950 9250 3000 9250
@@
 	2950 9050 3400 9050
 Wire Wire Line
-	1550 7100 1550 7000
-Wire Wire Line
-	1450 7100 1550 7100
-Wire Wire Line
-	1450 7000 1450 6900
+	1300 7100 1400 7100
+Wire Wire Line
+	1300 6900 1300 6800
 Wire Wire Line
 	2950 8950 2950 8850
@@
 L R R5
 U 1 1 54764F8C
-P 2000 6950
-F 0 "R5" V 2080 6950 40  0000 C CNN
-F 1 "10k" V 2007 6951 40  0000 C CNN
-F 2 "~" V 1930 6950 30  0000 C CNN
-F 3 "~" H 2000 6950 30  0000 C CNN
-	1    2000 6950
-	1    0    0    -1
-$EndComp
-Text GLabel 2250 7300 2    60   Input ~ 0
+P 2050 6950
+F 0 "R5" V 2130 6950 40  0000 C CNN
+F 1 "10k" V 2057 6951 40  0000 C CNN
+F 2 "~" V 1980 6950 30  0000 C CNN
+F 3 "~" H 2050 6950 30  0000 C CNN
+	1    2050 6950
+	1    0    0    -1
+$EndComp
+Text GLabel 2300 7300 2    60   Input ~ 0
 GPIO_A
-Text GLabel 2250 7400 2    60   Input ~ 0
+Text GLabel 2300 7400 2    60   Input ~ 0
 GPIO_B
 $Comp
 L R R6
 U 1 1 54764FA1
-P 2150 6950
-F 0 "R6" V 2230 6950 40  0000 C CNN
-F 1 "10k" V 2157 6951 40  0000 C CNN
-F 2 "~" V 2080 6950 30  0000 C CNN
-F 3 "~" H 2150 6950 30  0000 C CNN
-	1    2150 6950
+P 2200 6950
+F 0 "R6" V 2280 6950 40  0000 C CNN
+F 1 "10k" V 2207 6951 40  0000 C CNN
+F 2 "~" V 2130 6950 30  0000 C CNN
+F 3 "~" H 2200 6950 30  0000 C CNN
+	1    2200 6950
 	1    0    0    -1
 $EndComp
@@
 L R R3
 U 1 1 54764FBA
-P 1850 6950
-F 0 "R3" V 1930 6950 40  0000 C CNN
-F 1 "10k" V 1857 6951 40  0000 C CNN
-F 2 "~" V 1780 6950 30  0000 C CNN
-F 3 "~" H 1850 6950 30  0000 C CNN
-	1    1850 6950
-	1    0    0    -1
-$EndComp
-Wire Wire Line
-	1850 7200 1850 7300
-Connection ~ 1850 7300
-Wire Wire Line
-	2000 7200 2000 7400
-Connection ~ 2000 7400
-Wire Wire Line
-	2150 7200 2150 7500
-Connection ~ 2150 7500
+P 1900 6950
+F 0 "R3" V 1980 6950 40  0000 C CNN
+F 1 "10k" V 1907 6951 40  0000 C CNN
+F 2 "~" V 1830 6950 30  0000 C CNN
+F 3 "~" H 1900 6950 30  0000 C CNN
+	1    1900 6950
+	1    0    0    -1
+$EndComp
+Wire Wire Line
+	1900 7200 1900 7300
+Connection ~ 1900 7300
+Wire Wire Line
+	2050 7200 2050 7400
+Connection ~ 2050 7400
+Wire Wire Line
+	2200 7200 2200 7500
+Connection ~ 2200 7500
 $Comp
 L +5V_protected #PWR16
 U 1 1 547654F8
-P 2000 6600
-F 0 "#PWR16" H 2000 6690 20  0001 C CNN
-F 1 "+5V_protected" H 2000 6690 30  0000 C CNN
-F 2 "" H 2000 6600 60  0000 C CNN
-F 3 "" H 2000 6600 60  0000 C CNN
-	1    2000 6600
-	1    0    0    -1
-$EndComp
-Wire Wire Line
-	1850 6700 1850 6650
-Wire Wire Line
-	1850 6650 2150 6650
-Wire Wire Line
-	2150 6650 2150 6700
-Wire Wire Line
-	2000 6600 2000 6700
-Connection ~ 2000 6650
+P 2050 6600
+F 0 "#PWR16" H 2050 6690 20  0001 C CNN
+F 1 "+5V_protected" H 2050 6690 30  0000 C CNN
+F 2 "" H 2050 6600 60  0000 C CNN
+F 3 "" H 2050 6600 60  0000 C CNN
+	1    2050 6600
+	1    0    0    -1
+$EndComp
+Wire Wire Line
+	1900 6700 1900 6650
+Wire Wire Line
+	1900 6650 2200 6650
+Wire Wire Line
+	2200 6650 2200 6700
+Wire Wire Line
+	2050 6600 2050 6700
+Connection ~ 2050 6650
 $Comp
 L CONN_6 P2
@@
 L CONN_7 P3
 U 1 1 54788056
-P 1100 7300
-F 0 "P3" V 1070 7300 60  0000 C CNN
-F 1 "GPIO" V 1170 7300 60  0000 C CNN
-F 2 "~" H 1100 7300 60  0000 C CNN
-F 3 "~" H 1100 7300 60  0000 C CNN
-	1    1100 7300
+P 950 7200
+F 0 "P3" V 920 7200 60  0000 C CNN
+F 1 "GPIO" V 1020 7200 60  0000 C CNN
+F 2 "~" H 950 7200 60  0000 C CNN
+F 3 "~" H 950 7200 60  0000 C CNN
+	1    950  7200
 	-1   0    0    1
 $EndComp
@@
 L GND #PWR12
 U 1 1 54788074
-P 1650 7250
-F 0 "#PWR12" H 1650 7250 30  0001 C CNN
-F 1 "GND" H 1650 7180 30  0001 C CNN
-F 2 "" H 1650 7250 60  0000 C CNN
-F 3 "" H 1650 7250 60  0000 C CNN
-	1    1650 7250
-	1    0    0    -1
-$EndComp
-Wire Wire Line
-	1650 7250 1650 7200
-Wire Wire Line
-	1650 7200 1450 7200
+P 1500 7050
+F 0 "#PWR12" H 1500 7050 30  0001 C CNN
+F 1 "GND" H 1500 6980 30  0001 C CNN
+F 2 "" H 1500 7050 60  0000 C CNN
+F 3 "" H 1500 7050 60  0000 C CNN
+	1    1500 7050
+	1    0    0    -1
+$EndComp
+Wire Wire Line
+	1500 7050 1500 7000
+Wire Wire Line
+	1500 7000 1300 7000
 Connection ~ 12750 5150
 Wire Wire Line
@@
 	13850 4500 12750 4500
 Connection ~ 12750 4500
+Wire Wire Line
+	1400 7100 1400 6950
+Wire Wire Line
+	1350 7200 1300 7200
 $EndSCHEMATC

Commit message: routing
Parts:
- added C19: 100nF (DNP), ~, symbol C
Connections:
- wire segments 179 -> 181
Changed lines of the file:
@@
 $EndComp
 $Comp
-L GND #PWR10
+L GND #PWR11
 U 1 1 5454D86B
 P 1500 3000
-F 0 "#PWR10" H 1500 3000 30  0001 C CNN
+F 0 "#PWR11" H 1500 3000 30  0001 C CNN
 F 1 "GND" H 1500 2930 30  0001 C CNN
 F 2 "" H 1500 3000 60  0000 C CNN
@@
 $EndComp
 $Comp
-L +3.3V #PWR9
+L +3.3V #PWR10
 U 1 1 5454D884
 P 1450 8700
-F 0 "#PWR9" H 1450 8660 30  0001 C CNN
+F 0 "#PWR10" H 1450 8660 30  0001 C CNN
 F 1 "+3.3V" H 1450 8810 30  0000 C CNN
 F 2 "" H 1450 8700 60  0001 C CNN
@@
 $EndComp
 $Comp
-L GND #PWR42
+L GND #PWR44
 U 1 1 5454D8F7
 P 10850 4250
-F 0 "#PWR42" H 10850 4250 30  0001 C CNN
+F 0 "#PWR44" H 10850 4250 30  0001 C CNN
 F 1 "GND" H 10850 4180 30  0001 C CNN
 F 2 "" H 10850 4250 60  0001 C CNN
@@
 $EndComp
 $Comp
-L GND #PWR44
+L GND #PWR46
 U 1 1 5454D8F8
 P 12350 4250
-F 0 "#PWR44" H 12350 4250 30  0001 C CNN
+F 0 "#PWR46" H 12350 4250 30  0001 C CNN
 F 1 "GND" H 12350 4180 30  0001 C CNN
 F 2 "" H 12350 4250 60  0001 C CNN
@@
 $EndComp
 $Comp
-L GND #PWR40
+L GND #PWR42
 U 1 1 5454D8FE
 P 10500 4250
-F 0 "#PWR40" H 10500 4250 30  0001 C CNN
+F 0 "#PWR42" H 10500 4250 30  0001 C CNN
 F 1 "GND" H 10500 4180 30  0001 C CNN
 F 2 "" H 10500 4250 60  0001 C CNN
@@
 $EndComp
 $Comp
-L GND #PWR51
+L GND #PWR53
 U 1 1 5454D904
 P 14800 4250
-F 0 "#PWR51" H 14800 4250 30  0001 C CNN
+F 0 "#PWR53" H 14800 4250 30  0001 C CNN
 F 1 "GND" H 14800 4180 30  0001 C CNN
 F 2 "" H 14800 4250 60  0001 C CNN
@@
 $EndComp
 $Comp
-L GND #PWR46
+L GND #PWR48
 U 1 1 5454D909
 P 12950 4250
-F 0 "#PWR46" H 12950 4250 30  0001 C CNN
+F 0 "#PWR48" H 12950 4250 30  0001 C CNN
 F 1 "GND" H 12950 4180 30  0001 C CNN
 F 2 "" H 12950 4250 60  0001 C CNN
@@
 $EndComp
 $Comp
-L GND #PWR49
+L GND #PWR51
 U 1 1 5454D90A
 P 14450 4250
-F 0 "#PWR49" H 14450 4250 30  0001 C CNN
+F 0 "#PWR51" H 14450 4250 30  0001 C CNN
 F 1 "GND" H 14450 4180 30  0001 C CNN
 F 2 "" H 14450 4250 60  0001 C CNN
@@
 $EndComp
 $Comp
-L GND #PWR7
+L GND #PWR8
 U 1 1 5454DBE8
 P 1400 1450
-F 0 "#PWR7" H 1400 1450 30  0001 C CNN
+F 0 "#PWR8" H 1400 1450 30  0001 C CNN
 F 1 "GND" H 1400 1380 30  0001 C CNN
 F 2 "" H 1400 1450 60  0000 C CNN
@@
 $EndComp
 $Comp
-L +3.3V #PWR18
+L +3.3V #PWR17
 U 1 1 5454EDA2
 P 2050 2300
-F 0 "#PWR18" H 2050 2260 30  0001 C CNN
+F 0 "#PWR17" H 2050 2260 30  0001 C CNN
 F 1 "+3.3V" H 2050 2410 30  0000 C CNN
 F 2 "" H 2050 2300 60  0000 C CNN
@@
 $EndComp
 $Comp
-L GND #PWR48
+L GND #PWR50
 U 1 1 545A9ED6
 P 14350 6450
-F 0 "#PWR48" H 14350 6450 30  0001 C CNN
+F 0 "#PWR50" H 14350 6450 30  0001 C CNN
 F 1 "GND" H 14350 6380 30  0001 C CNN
 F 2 "" H 14350 6450 60  0000 C CNN
@@
 $EndComp
 $Comp
-L GND #PWR43
+L GND #PWR45
 U 1 1 545AAF07
 P 12250 6550
-F 0 "#PWR43" H 12250 6550 30  0001 C CNN
+F 0 "#PWR45" H 12250 6550 30  0001 C CNN
 F 1 "GND" H 12250 6480 30  0001 C CNN
 F 2 "" H 12250 6550 60  0000 C CNN
@@
 $EndComp
 $Comp
-L +9V #PWR41
+L +9V #PWR43
 U 1 1 545AB10D
 P 10750 2850
-F 0 "#PWR41" H 10750 2820 20  0001 C CNN
+F 0 "#PWR43" H 10750 2820 20  0001 C CNN
 F 1 "+9V" H 10750 2960 30  0000 C CNN
 F 2 "" H 10750 2850 60  0000 C CNN
@@
 $EndComp
 $Comp
-L +9V #PWR50
+L +9V #PWR52
 U 1 1 545AB11A
 P 14550 2800
-F 0 "#PWR50" H 14550 2770 20  0001 C CNN
+F 0 "#PWR52" H 14550 2770 20  0001 C CNN
 F 1 "+9V" H 14550 2900 30  0000 C CNN
 F 2 "" H 14550 2800 60  0000 C CNN
@@
 $EndComp
 $Comp
-L GND #PWR17
+L GND #PWR16
 U 1 1 545F8B91
 P 2000 8950
-F 0 "#PWR17" H 2000 8950 30  0001 C CNN
+F 0 "#PWR16" H 2000 8950 30  0001 C CNN
 F 1 "GND" H 2000 8880 30  0001 C CNN
 F 2 "" H 2000 8950 60  0001 C CNN
@@
 NoConn ~ 1050 1100
 $Comp
-L +BATT #PWR45
+L +BATT #PWR47
 U 1 1 5464BE5C
 P 12650 2750
-F 0 "#PWR45" H 12650 2700 20  0001 C CNN
+F 0 "#PWR47" H 12650 2700 20  0001 C CNN
 F 1 "+BATT" H 12650 2850 30  0000 C CNN
 F 2 "" H 12650 2750 60  0000 C CNN
@@
 $EndComp
 $Comp
-L +3.3V_A #PWR47
+L +3.3V_A #PWR49
 U 1 1 5464C46E
 P 13700 5450
-F 0 "#PWR47" H 13700 5410 30  0001 C CNN
+F 0 "#PWR49" H 13700 5410 30  0001 C CNN
 F 1 "+3.3V_A" H 13700 5560 30  0000 C CNN
 F 2 "" H 13700 5450 60  0000 C CNN
@@
 $EndComp
 $Comp
-L +3.3V_A #PWR52
+L +3.3V_A #PWR54
 U 1 1 5464C47E
 P 15000 5600
-F 0 "#PWR52" H 15000 5560 30  0001 C CNN
+F 0 "#PWR54" H 15000 5560 30  0001 C CNN
 F 1 "+3.3V_A" H 15000 5710 30  0000 C CNN
 F 2 "" H 15000 5600 60  0000 C CNN
@@
 GPIO_ADC
 $Comp
-L +3.3V_A #PWR11
+L +3.3V_A #PWR9
 U 1 1 5464C7D0
 P 1400 6950
-F 0 "#PWR11" H 1400 6910 30  0001 C CNN
+F 0 "#PWR9" H 1400 6910 30  0001 C CNN
 F 1 "+3.3V_A" H 1400 7060 30  0000 C CNN
 F 2 "" H 1400 6950 60  0000 C CNN
@@
 $EndComp
 $Comp
-L +5V_protected #PWR8
+L +5V_protected #PWR7
 U 1 1 5464CB8A
 P 1300 6800
-F 0 "#PWR8" H 1300 6890 20  0001 C CNN
+F 0 "#PWR7" H 1300 6890 20  0001 C CNN
 F 1 "+5V_protected" H 1300 6890 30  0000 C CNN
 F 2 "" H 1300 6800 60  0000 C CNN
@@
 Connection ~ 2200 7500
 $Comp
-L +5V_protected #PWR16
+L +5V_protected #PWR18
 U 1 1 547654F8
 P 2050 6600
-F 0 "#PWR16" H 2050 6690 20  0001 C CNN
+F 0 "#PWR18" H 2050 6690 20  0001 C CNN
 F 1 "+5V_protected" H 2050 6690 30  0000 C CNN
 F 2 "" H 2050 6600 60  0000 C CNN
@@
 Wire Wire Line
 	1350 7200 1300 7200
+$Comp
+L C C19
+U 1 1 547F68F0
+P 10150 2450
+F 0 "C19" H 10150 2550 40  0000 L CNN
+F 1 "100nF (DNP)" V 10300 2350 40  0000 L CNN
+F 2 "~" H 10188 2300 30  0000 C CNN
+F 3 "~" H 10150 2450 60  0000 C CNN
+	1    10150 2450
+	-1   0    0    1
+$EndComp
+$Comp
+L +9V #PWR40
+U 1 1 547F68FD
+P 10150 2200
+F 0 "#PWR40" H 10150 2170 20  0001 C CNN
+F 1 "+9V" H 10150 2310 30  0000 C CNN
+F 2 "" H 10150 2200 60  0000 C CNN
+F 3 "" H 10150 2200 60  0000 C CNN
+	1    10150 2200
+	1    0    0    -1
+$EndComp
+$Comp
+L GND #PWR41
+U 1 1 547F6905
+P 10150 2750
+F 0 "#PWR41" H 10150 2750 30  0001 C CNN
+F 1 "GND" H 10150 2680 30  0001 C CNN
+F 2 "" H 10150 2750 60  0000 C CNN
+F 3 "" H 10150 2750 60  0000 C CNN
+	1    10150 2750
+	1    0    0    -1
+$EndComp
+Wire Wire Line
+	10150 2200 10150 2250
+Wire Wire Line
+	10150 2650 10150 2750
 $EndSCHEMATC

Commit message: routing, changed connectors
Changed lines of the file:
@@
 Sheet 1 1
 Title "Motor control board"
-Date "4 dec 2014"
+Date "6 dec 2014"
 Rev "V00"
 Comp "CVRA"
@@
 	-1   0    0    1
 $EndComp
-Text GLabel 3000 9150 2    60   Input ~ 0
+Text GLabel 3000 9250 2    60   Input ~ 0
 CANL
 Text GLabel 2300 7500 2    60   Input ~ 0
@@
 Text Notes 12700 6250 0    60   ~ 0
 Fc = 4.8kHz
-Text GLabel 3000 9250 2    60   Input ~ 0
+Text GLabel 3000 9150 2    60   Input ~ 0
 CANH
 Wire Wire Line

Commit message: resistive divider values & schematic annotations
Parts:
- C18: value C -> 10nF
- R12: value R -> 100k
- R13: value R -> 18k
Other:
- note added: "3s-4s Lipo\n(9-16.8V)"
- note added: "8.6V"
- note added: "[Uin (max) = 16.8V, Uadc max = 3.3V]\nGain K = R13/R12+R13 = 0.1525 (-> 21.5V abs. max)\nFc = 1/K*R12*C18*2pi = 1kHz"
Changed lines of the file:
@@
 Sheet 1 1
 Title "Motor control board"
-Date "6 dec 2014"
+Date "3 jan 2015"
 Rev "V00"
 Comp "CVRA"
@@
 P 4150 1200
 F 0 "R12" V 4230 1200 40  0000 C CNN
-F 1 "R" V 4157 1201 40  0000 C CNN
+F 1 "100k" V 4157 1201 40  0000 C CNN
 F 2 "~" V 4080 1200 30  0000 C CNN
 F 3 "~" H 4150 1200 30  0000 C CNN
@@
 P 4150 1800
 F 0 "R13" V 4230 1800 40  0000 C CNN
-F 1 "R" V 4157 1801 40  0000 C CNN
+F 1 "18k" V 4157 1801 40  0000 C CNN
 F 2 "~" V 4080 1800 30  0000 C CNN
 F 3 "~" H 4150 1800 30  0000 C CNN
@@
 P 3950 1800
 F 0 "C18" H 3950 1900 40  0000 L CNN
-F 1 "C" H 3956 1715 40  0000 L CNN
+F 1 "10nF" H 3956 1715 40  0000 L CNN
 F 2 "~" H 3988 1650 30  0000 C CNN
 F 3 "~" H 3950 1800 60  0000 C CNN
@@
 Wire Wire Line
 	10150 2650 10150 2750
+Text Notes 4350 1700 0    40   ~ 0
+[Uin (max) = 16.8V, Uadc max = 3.3V]\nGain K = R13/R12+R13 = 0.1525 (-> 21.5V abs. max)\nFc = 1/K*R12*C18*2pi = 1kHz
+Text Notes 2900 5450 0    60   ~ 0
+3s-4s Lipo\n(9-16.8V)
+Text Notes 2350 1000 0    60   ~ 0
+8.6V
 $EndSCHEMATC

Commit message: fix current amplifier common mode issue
Connections:
- net labels removed: +5V_PROTECTED
- wire segments 181 -> 183
Other:
- moved on the sheet: C14, C15, C16, C19, D3, D4, IC4, IC5, IC6, Q1, Q2, Q3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
